File: block.kicad_sch (KiCad schematic)
At the start: 12 parts

Commit message: Save progress
Parts:
- renumbered C43 to C73, C44 to C74, C51 to C75, C47 to C76, C50 to C77, R41 to R69, R42 to R70, R43 to R71, R44 to R72, R45 to R73, R46 to R74, R47 to R75
Changed lines of the file:
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@@
 		(dnp no)
 		(fields_autoplaced yes)
-		(property "Reference" "C43"
+		(property "Reference" "C73"
 			(at 110.49 86.3599 0)
 			(effects
@@
 		(dnp no)
 		(fields_autoplaced yes)
-		(property "Reference" "C44"
+		(property "Reference" "C74"
 			(at 123.19 86.3599 0)
 			(effects
@@
 		(dnp no)
 		(fields_autoplaced yes)
-		(property "Reference" "R47"
+		(property "Reference" "R75"
 			(at 100.33 130.81 90)
 			(effects
@@
 		(dnp no)
 		(fields_autoplaced yes)
-		(property "Reference" "R46"
+		(property "Reference" "R74"
 			(at 100.33 120.65 90)
 			(effects
@@
 		(dnp no)
 		(fields_autoplaced yes)
-		(property "Reference" "R41"
+		(property "Reference" "R69"
 			(at 100.33 64.77 90)
 			(effects
@@
 		(dnp no)
 		(fields_autoplaced yes)
-		(property "Reference" "C47"
+		(property "Reference" "C76"
 			(at 110.49 119.3799 0)
 			(effects
@@
 		(dnp no)
 		(fields_autoplaced yes)
-		(property "Reference" "R43"
+		(property "Reference" "R71"
 			(at 100.33 87.63 90)
 			(effects
@@
 		(dnp no)
 		(fields_autoplaced yes)
-		(property "Reference" "R44"
+		(property "Reference" "R72"
 			(at 100.33 97.79 90)
 			(effects
@@
 		(dnp no)
 		(fields_autoplaced yes)
-		(property "Reference" "C51"
+		(property "Reference" "C75"
 			(at 135.89 109.2199 0)
 			(effects
@@
 		(dnp no)
 		(fields_autoplaced yes)
-		(property "Reference" "C50"
+		(property "Reference" "C77"
 			(at 123.19 119.3799 0)
 			(effects
@@
 		(dnp no)
 		(fields_autoplaced yes)
-		(property "Reference" "#PWR033"
+		(property "Reference" "#PWR045"
 			(at 132.08 123.19 0)
 			(effects
@@
 		(dnp no)
 		(fields_autoplaced yes)
-		(property "Reference" "R42"
+		(property "Reference" "R70"
 			(at 100.33 74.93 90)
 			(effects
@@
 		(dnp no)
 		(fields_autoplaced yes)
-		(property "Reference" "R45"
+		(property "Reference" "R73"
 			(at 100.33 107.95 90)
 			(effects
