File: filter.kicad_sch (KiCad schematic)
At the start: 2 parts

Commit message: Save progress
Parts:
- renumbered C1 to C8, R1 to R8
Changed lines of the file:
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@@
 		(dnp no)
 		(fields_autoplaced yes)
-		(property "Reference" "C1"
+		(property "Reference" "C8"
 			(at 93.98 68.5799 0)
 			(effects
@@
 		(dnp no)
 		(fields_autoplaced yes)
-		(property "Reference" "#PWR03"
+		(property "Reference" "#PWR053"
 			(at 90.17 82.55 0)
 			(effects
@@
 		(dnp no)
 		(fields_autoplaced yes)
-		(property "Reference" "R1"
+		(property "Reference" "R8"
 			(at 83.82 57.15 90)
 			(effects
