File: transceiver.kicad_sch (KiCad schematic)
At the start: 15 parts, among them J3 Conn_01x02_Pin

Commit message: Save progress
Parts:
- renumbered C14 to C18, C17 to C19, C15 to C20, D2 to D3, R18 to R22, R16 to R24, R20 to R26
Changed lines of the file:
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@@
 		(on_board yes)
 		(dnp no)
-		(property "Reference" "#PWR014"
+		(property "Reference" "#PWR017"
 			(at 110.49 73.66 0)
 			(effects
@@
 		(dnp no)
 		(fields_autoplaced yes)
-		(property "Reference" "R18"
+		(property "Reference" "R22"
 			(at 91.44 66.0399 0)
 			(effects
@@
 		(dnp no)
 		(fields_autoplaced yes)
-		(property "Reference" "#PWR012"
+		(property "Reference" "#PWR016"
 			(at 69.85 52.07 0)
 			(effects
@@
 		(dnp no)
 		(fields_autoplaced yes)
-		(property "Reference" "#PWR013"
+		(property "Reference" "#PWR019"
 			(at 69.85 92.71 0)
 			(effects
@@
 		(dnp no)
 		(fields_autoplaced yes)
-		(property "Reference" "C15"
+		(property "Reference" "C20"
 			(at 97.79 66.04 90)
 			(effects
@@
 		(dnp no)
 		(fields_autoplaced yes)
-		(property "Reference" "#PWR011"
+		(property "Reference" "#PWR015"
 			(at 50.8 52.07 0)
 			(effects
@@
 		(dnp no)
 		(fields_autoplaced yes)
-		(property "Reference" "D2"
+		(property "Reference" "D3"
 			(at 72.39 63.4999 90)
 			(effects
@@
 		(dnp no)
 		(fields_autoplaced yes)
-		(property "Reference" "C14"
+		(property "Reference" "C18"
 			(at 54.61 63.4999 0)
 			(effects
@@
 		(on_board yes)
 		(dnp no)
-		(property "Reference" "R16"
+		(property "Reference" "R24"
 			(at 63.5 76.962 90)
 			(effects
@@
 		(dnp no)
 		(fields_autoplaced yes)
-		(property "Reference" "R20"
+		(property "Reference" "R26"
 			(at 97.79 80.01 90)
 			(effects
@@
 		(on_board yes)
 		(dnp no)
-		(property "Reference" "C17"
+		(property "Reference" "C19"
 			(at 130.81 63.5 90)
 			(effects
